File: REV 0-2 PCB/FlatPack 0-2/Buck Converter SubBoard 0-2/Buck Converter SubBoard 0-2/Buck Converter SubBoard 0-2.sch (KiCad schematic (older format))
At the start: 12 parts

Commit message: Pushing Buck Converter Sub Board for 0-2
Parts:
- added C6, C8: 100n, Capacitor_SMD:C_0603_1608Metric_Pad1.05x0.95mm_HandSolder, symbol Device:C
- added C7: 4u7, Capacitor_SMD:C_0805_2012Metric_Pad1.15x1.40mm_HandSolder, symbol Device:C
- added D2, D3: RED, LED_SMD:LED_0603_1608Metric_Pad1.05x0.95mm_HandSolder, symbol Device:LED
- added D4: 1N4448, Diode_SMD:D_SOD-123, symbol Device:D
- added J1: Conn_01x04, Connector_PinHeader_2.54mm:PinHeader_1x04_P2.54mm_Vertical, symbol Connector_Generic:Conn_01x04
- added J2: Conn_02x07_Odd_Even, Connector_PinHeader_2.54mm:PinHeader_2x07_P2.54mm_Vertical, symbol Connector_Generic:Conn_02x07_Odd_Even
- added R1: 1k, Resistor_SMD:R_0603_1608Metric_Pad1.05x0.95mm_HandSolder, symbol Device:R
- added R6: 390R, Resistor_SMD:R_0603_1608Metric_Pad1.05x0.95mm_HandSolder, symbol Device:R
- added R7: 120R, Resistor_SMD:R_0603_1608Metric_Pad1.05x0.95mm_HandSolder, symbol Device:R
- added TP1, TP2, TP3, TP4, TP5, TP6, TP7, TP8, TP9: TestPoint_Probe, TestPoint:TestPoint_Keystone_5000-5004_Miniature, symbol Connector:TestPoint_Probe
- added U2: ZLDO1117-33, Package_TO_SOT_SMD:TO-252-2, symbol Regulator_Linear:AP1117-33
- C1, C2: renamed from C?; value C -> 1u; footprint (none) -> Capacitor_SMD:C_0805_2012Metric_Pad1.15x1.40mm_HandSolder
- C3: renamed from C?; value C -> 100n; footprint (none) -> Capacitor_SMD:C_0603_1608Metric_Pad1.05x0.95mm_HandSolder
- C4, C5: renamed from C?; value C -> 4u7; footprint (none) -> Capacitor_SMD:C_0805_2012Metric_Pad1.15x1.40mm_HandSolder
- D1: renamed from D?; footprint (none) -> Diode_SMD:D_SOD-123
- L1: renamed from L?; value L -> 47uH; footprint (none) -> Inductor_SMD:L_Taiyo-Yuden_NR-40xx_HandSoldering
- R2, R5: renamed from R?; value R -> 10k; footprint (none) -> Resistor_SMD:R_0603_1608Metric_Pad1.05x0.95mm_HandSolder
- R3: renamed from R?; value R -> 30k; footprint (none) -> Resistor_SMD:R_0603_1608Metric_Pad1.05x0.95mm_HandSolder
- R4: renamed from R?; value R -> 390R; footprint (none) -> Resistor_SMD:R_0603_1608Metric_Pad1.05x0.95mm_HandSolder
- gave numbers to parts that had none: 1
Connections:
- net labels added: +3.3V, +5V, GND, VBUS
- wire segments 22 -> 109
