File: REV 0-1 PCB/Kicad Files/AFE.sch (KiCad schematic (older format))
At the start: 143 parts, among them Q1 RUC002N05HZGT116, Q10 RUC002N05HZGT116, Q11 IPD60N10S4L-12, Q12 RUC002N05HZGT116, Q2 RUC002N05HZGT116, Q3 RUC002N05HZGT116, Q4 RUC002N05HZGT116, Q5 RUC002N05HZGT116, Q6 RUC002N05HZGT116, Q7 RUC002N05HZGT116, Q8 RUC002N05HZGT116, Q9 RUC002N05HZGT116, U1 BQ76930

Commit message: Fixing working tree, pushing a bunch of SubBoards and FlatPack BOM
Parts:
- Q1, Q10, Q12, Q2, Q3, Q4, Q5, Q6, Q7, Q8, Q9: symbol Transistor_FET:RUC002N05HZGT116 -> FusIon-Pack-rescue:RUC002N05HZGT116-Transistor_FET
- Q11: symbol Transistor_FET:IPD60N10S4L-12 -> FusIon-Pack-rescue:IPD60N10S4L-12-Transistor_FET
- U1: symbol Battery_Management:BQ76930 -> FusIon-Pack-rescue:BQ76930-Battery_Management
Changed lines of the file:
@@
 EESchema Schematic File Version 4
 LIBS:FusIon Pack-cache
-EELAYER 26 0
+EELAYER 29 0
 EELAYER END
 $Descr A4 8268 11693 portrait
@@
 $EndDescr
 $Comp
-L Battery_Management:BQ76930 U1
+L FusIon-Pack-rescue:BQ76930-Battery_Management U1
 U 1 1 5C410908
 P 5700 5400
@@
 $EndComp
 $Comp
-L Transistor_FET:RUC002N05HZGT116 Q1
+L FusIon-Pack-rescue:RUC002N05HZGT116-Transistor_FET Q1
 U 1 1 5C41189A
 P 2300 1350
@@
 Connection ~ 2850 1350
 $Comp
-L Transistor_FET:RUC002N05HZGT116 Q2
+L FusIon-Pack-rescue:RUC002N05HZGT116-Transistor_FET Q2
 U 1 1 5C4381FC
 P 2300 2400
@@
 Connection ~ 2850 2400
 $Comp
-L Transistor_FET:RUC002N05HZGT116 Q3
+L FusIon-Pack-rescue:RUC002N05HZGT116-Transistor_FET Q3
 U 1 1 5C438D03
 P 2300 3450
@@
 Connection ~ 2850 3450
 $Comp
-L Transistor_FET:RUC002N05HZGT116 Q4
+L FusIon-Pack-rescue:RUC002N05HZGT116-Transistor_FET Q4
 U 1 1 5C438D55
 P 2300 4500
@@
 Connection ~ 2850 4500
 $Comp
-L Transistor_FET:RUC002N05HZGT116 Q5
+L FusIon-Pack-rescue:RUC002N05HZGT116-Transistor_FET Q5
 U 1 1 5C43B02B
 P 2300 5550
@@
 Connection ~ 2200 5250
 $Comp
-L Transistor_FET:RUC002N05HZGT116 Q6
+L FusIon-Pack-rescue:RUC002N05HZGT116-Transistor_FET Q6
 U 1 1 5C43B07D
 P 2300 6600
@@
 Connection ~ 2850 6600
 $Comp
-L Transistor_FET:RUC002N05HZGT116 Q7
+L FusIon-Pack-rescue:RUC002N05HZGT116-Transistor_FET Q7
 U 1 1 5C43B0CF
 P 2300 7650
@@
 Connection ~ 2850 7650
 $Comp
-L Transistor_FET:RUC002N05HZGT116 Q8
+L FusIon-Pack-rescue:RUC002N05HZGT116-Transistor_FET Q8
 U 1 1 5C43B121
 P 2300 8700
@@
 Connection ~ 2850 8700
 $Comp
-L Transistor_FET:RUC002N05HZGT116 Q9
+L FusIon-Pack-rescue:RUC002N05HZGT116-Transistor_FET Q9
 U 1 1 5C44320B
 P 2300 9750
@@
 Connection ~ 2850 9750
 $Comp
-L Transistor_FET:RUC002N05HZGT116 Q10
+L FusIon-Pack-rescue:RUC002N05HZGT116-Transistor_FET Q10
 U 1 1 5C44325D
 P 2300 10800
@@
 REGOUT
 $Comp
-L Transistor_FET:IPD60N10S4L-12 Q11
+L FusIon-Pack-rescue:IPD60N10S4L-12-Transistor_FET Q11
 U 1 1 5CEE5B76
 P 5600 2250
@@
 $EndComp
 $Comp
-L Transistor_FET:RUC002N05HZGT116 Q12
+L FusIon-Pack-rescue:RUC002N05HZGT116-Transistor_FET Q12
 U 1 1 5C6A21AD
 P 5600 9300
