File: REV 0-1 PCB/Kicad Files/Boost_Charger.sch (KiCad schematic (older format))
At the start: 69 parts, among them Q18 RUC002N05HZGT116, Q19 DMPH6050SK3, Q20 IPD60N10S4L-12, Q21 RUC002N05HZGT116, Q22 DMPH6050SK3, Q23 DMPH6050SK3, U7 ZXCT108x, U8 LTC3783, U9 ZXCT108x

Commit message: Fixing working tree, pushing a bunch of SubBoards and FlatPack BOM
Parts:
- Q18, Q21: symbol Transistor_FET:RUC002N05HZGT116 -> FusIon-Pack-rescue:RUC002N05HZGT116-Transistor_FET
- Q19, Q22, Q23: symbol Transistor_FET:IRF5210 -> FusIon-Pack-rescue:IRF5210-Transistor_FET
- Q20: symbol Transistor_FET:IPD60N10S4L-12 -> FusIon-Pack-rescue:IPD60N10S4L-12-Transistor_FET
- U7, U9: symbol Amplifier_Current:ZXCT108x -> FusIon-Pack-rescue:ZXCT108x-Amplifier_Current
- U8: symbol Regulator_Controller:LTC3783 -> FusIon-Pack-rescue:LTC3783-Regulator_Controller
Changed lines of the file:
@@
 EESchema Schematic File Version 4
 LIBS:FusIon Pack-cache
-EELAYER 26 0
+EELAYER 29 0
 EELAYER END
 $Descr A4 11693 8268
@@
 $EndDescr
 $Comp
-L Regulator_Controller:LTC3783 U8
+L FusIon-Pack-rescue:LTC3783-Regulator_Controller U8
 U 1 1 5CD3D89B
 P 4750 4300
@@
 	5700 4600 5700 4800
 $Comp
-L Transistor_FET:IPD60N10S4L-12 Q20
+L FusIon-Pack-rescue:IPD60N10S4L-12-Transistor_FET Q20
 U 1 1 5C4D1E56
 P 6050 4000
@@
 I_SET
 $Comp
-L Transistor_FET:RUC002N05HZGT116 Q21
+L FusIon-Pack-rescue:RUC002N05HZGT116-Transistor_FET Q21
 U 1 1 5C5090B8
 P 8550 4700
@@
 Connection ~ 2850 4100
 $Comp
-L Transistor_FET:IRF5210 Q19
+L FusIon-Pack-rescue:IRF5210-Transistor_FET Q19
 U 1 1 5C553EA6
 P 2600 3450
@@
 	2600 3700 2600 3650
 $Comp
-L Transistor_FET:RUC002N05HZGT116 Q18
+L FusIon-Pack-rescue:RUC002N05HZGT116-Transistor_FET Q18
 U 1 1 5C569DD3
 P 2250 4550
@@
 BOOST_OUT
 $Comp
-L Amplifier_Current:ZXCT108x U7
+L FusIon-Pack-rescue:ZXCT108x-Amplifier_Current U7
 U 1 1 5C6744E0
 P 3900 2100
@@
 $EndComp
 $Comp
-L Amplifier_Current:ZXCT108x U9
+L FusIon-Pack-rescue:ZXCT108x-Amplifier_Current U9
 U 1 1 5C674814
 P 8200 2100
@@
 Connection ~ 5300 2750
 $Comp
-L Transistor_FET:IRF5210 Q23
+L FusIon-Pack-rescue:IRF5210-Transistor_FET Q23
 U 1 1 5C7A80D0
 P 9400 3250
@@
 $EndComp
 $Comp
-L Transistor_FET:IRF5210 Q22
+L FusIon-Pack-rescue:IRF5210-Transistor_FET Q22
 U 1 1 5C7A8572
 P 8650 3250
