File: REV 0-1 PCB/Kicad Files/CAN.sch (KiCad schematic (older format))
At the start: 10 parts, among them U5 ATA6561

Commit message: Fixing working tree, pushing a bunch of SubBoards and FlatPack BOM
Parts:
- U5: symbol Interface_CAN_LIN:ATA6561 -> FusIon-Pack-rescue:ATA6561-Interface_CAN_LIN
Changed lines of the file:
@@
 EESchema Schematic File Version 4
 LIBS:FusIon Pack-cache
-EELAYER 26 0
+EELAYER 29 0
 EELAYER END
 $Descr A4 11693 8268
@@
 $EndDescr
 $Comp
-L Interface_CAN_LIN:ATA6561 U5
+L FusIon-Pack-rescue:ATA6561-Interface_CAN_LIN U5
 U 1 1 5CBFEB3E
 P 5600 4150
