File: REV 0-1 PCB/Kicad Files/FLASH.sch (KiCad schematic (older format))
At the start: 3 parts, among them U6 W25Q16JVSSIQ

Commit message: Fixing working tree, pushing a bunch of SubBoards and FlatPack BOM
Parts:
- U6: symbol Memory_Flash:W25Q16JVSSIQ -> FusIon-Pack-rescue:W25Q16JVSSIQ-Memory_Flash
Changed lines of the file:
@@
 EESchema Schematic File Version 4
 LIBS:FusIon Pack-cache
-EELAYER 26 0
+EELAYER 29 0
 EELAYER END
 $Descr A4 11693 8268
@@
 $EndDescr
 $Comp
-L Memory_Flash:W25Q16JVSSIQ U6
+L FusIon-Pack-rescue:W25Q16JVSSIQ-Memory_Flash U6
 U 1 1 5CC0741A
 P 5800 4150
