File: REV 0-1 PCB/Kicad Files/FusIon Pack.sch (KiCad schematic (older format))
At the start: 42 parts, among them J1 USB_BOARD

Commit message: Fixing working tree, pushing a bunch of SubBoards and FlatPack BOM
Parts:
- BT1, BT10, BT2, BT3, BT4, BT5, BT6, BT7, BT8, BT9: symbol Device:Battery_Cell_Short -> FusIon-Pack-rescue:Battery_Cell_Short-Device
- F2, F3, F4, F5: symbol Graphic:Fiducial -> FusIon-Pack-rescue:Fiducial-Graphic
Changed lines of the file:
@@
 EESchema Schematic File Version 4
 LIBS:FusIon Pack-cache
-EELAYER 26 0
+EELAYER 29 0
 EELAYER END
 $Descr A4 11693 8268
@@
 	5050 5700 5550 5700
 $Comp
-L Device:Battery_Cell_Short BT10
+L FusIon-Pack-rescue:Battery_Cell_Short-Device BT10
 U 1 1 5C860E0C
 P 1650 5300
@@
 $EndComp
 $Comp
-L Device:Battery_Cell_Short BT9
+L FusIon-Pack-rescue:Battery_Cell_Short-Device BT9
 U 1 1 5C860F33
 P 1650 5000
@@
 $EndComp
 $Comp
-L Device:Battery_Cell_Short BT8
+L FusIon-Pack-rescue:Battery_Cell_Short-Device BT8
 U 1 1 5C860F74
 P 1650 4700
@@
 $EndComp
 $Comp
-L Device:Battery_Cell_Short BT7
+L FusIon-Pack-rescue:Battery_Cell_Short-Device BT7
 U 1 1 5C860F9E
 P 1650 4400
@@
 $EndComp
 $Comp
-L Device:Battery_Cell_Short BT6
+L FusIon-Pack-rescue:Battery_Cell_Short-Device BT6
 U 1 1 5C860FC8
 P 1650 4100
@@
 $EndComp
 $Comp
-L Device:Battery_Cell_Short BT5
+L FusIon-Pack-rescue:Battery_Cell_Short-Device BT5
 U 1 1 5C860FF4
 P 1650 3800
@@
 $EndComp
 $Comp
-L Device:Battery_Cell_Short BT4
+L FusIon-Pack-rescue:Battery_Cell_Short-Device BT4
 U 1 1 5C86101E
 P 1650 3500
@@
 $EndComp
 $Comp
-L Device:Battery_Cell_Short BT3
+L FusIon-Pack-rescue:Battery_Cell_Short-Device BT3
 U 1 1 5C86104E
 P 1650 3200
@@
 $EndComp
 $Comp
-L Device:Battery_Cell_Short BT2
+L FusIon-Pack-rescue:Battery_Cell_Short-Device BT2
 U 1 1 5C8610C4
 P 1650 2900
@@
 $EndComp
 $Comp
-L Device:Battery_Cell_Short BT1
+L FusIon-Pack-rescue:Battery_Cell_Short-Device BT1
 U 1 1 5C8610F4
 P 1650 2600
@@
 	3650 5500 5550 5500
 $Comp
-L Graphic:Fiducial F2
+L FusIon-Pack-rescue:Fiducial-Graphic F2
 U 1 1 5C71EC06
 P 1400 1150
@@
 $EndComp
 $Comp
-L Graphic:Fiducial F3
+L FusIon-Pack-rescue:Fiducial-Graphic F3
 U 1 1 5C71F01E
 P 1400 1300
@@
 $EndComp
 $Comp
-L Graphic:Fiducial F4
+L FusIon-Pack-rescue:Fiducial-Graphic F4
 U 1 1 5C71F068
 P 1400 1450
@@
 $EndComp
 $Comp
-L Graphic:Fiducial F5
+L FusIon-Pack-rescue:Fiducial-Graphic F5
 U 1 1 5C71F0B2
 P 1400 1600
