File: REV 0-1 PCB/Kicad Files/LED Header.sch (KiCad schematic (older format))
At the start: 9 parts, among them J3 B4B-XH-A(LF)(SN), Q17 RUC002N05HZGT116

Commit message: Fixing working tree, pushing a bunch of SubBoards and FlatPack BOM
Parts:
- Q17: symbol Transistor_FET:RUC002N05HZGT116 -> FusIon-Pack-rescue:RUC002N05HZGT116-Transistor_FET
Changed lines of the file:
@@
 EESchema Schematic File Version 4
 LIBS:FusIon Pack-cache
-EELAYER 26 0
+EELAYER 29 0
 EELAYER END
 $Descr A4 11693 8268
@@
 $EndComp
 $Comp
-L Transistor_FET:RUC002N05HZGT116 Q17
+L FusIon-Pack-rescue:RUC002N05HZGT116-Transistor_FET Q17
 U 1 1 5CC0E04D
 P 5600 5200
