File: REV 0-1 PCB/Kicad Files/LV_Regulation.sch (KiCad schematic (older format))
At the start: 22 parts, among them Q15 RUC002N05HZGT116, Q16 FQT5P10TF, U3 L7805, U4 AP2114H-3.3TRG1

Commit message: Pushing stuff for Rev II PCB
Parts:
- D43: value 6V2 -> 6.2V
Changed lines of the file:
@@
 P 4300 3700
 F 0 "D43" V 4254 3779 50  0000 L CNN
-F 1 "6V2" V 4345 3779 50  0000 L CNN
+F 1 "6.2V" V 4345 3779 50  0000 L CNN
 F 2 "Diode_SMD:D_SMA" H 4300 3700 50  0001 C CNN
 F 3 "~" H 4300 3700 50  0001 C CNN

Commit message: Fixing working tree, pushing a bunch of SubBoards and FlatPack BOM
Parts:
- Q15: symbol Transistor_FET:RUC002N05HZGT116 -> FusIon-Pack-rescue:RUC002N05HZGT116-Transistor_FET
- Q16: symbol Transistor_FET:FQT5P10TF -> FusIon-Pack-rescue:FQT5P10TF-Transistor_FET
Changed lines of the file:
@@
 EESchema Schematic File Version 4
 LIBS:FusIon Pack-cache
-EELAYER 26 0
+EELAYER 29 0
 EELAYER END
 $Descr A4 11693 8268
@@
 $EndDescr
 $Comp
-L Transistor_FET:FQT5P10TF Q16
+L FusIon-Pack-rescue:FQT5P10TF-Transistor_FET Q16
 U 1 1 5CBD378D
 P 4200 3300
@@
 $EndComp
 $Comp
-L Transistor_FET:RUC002N05HZGT116 Q15
+L FusIon-Pack-rescue:RUC002N05HZGT116-Transistor_FET Q15
 U 1 1 5CBD38B9
 P 3800 4300
