File: REV 0-1 PCB/Kicad Files/Output_Conn.sch (KiCad schematic (older format))
At the start: 5 parts, among them J4 Conn_01x05_Male, J5 XT60

Commit message: Fixing working tree, pushing a bunch of SubBoards and FlatPack BOM
Parts:
- J5: symbol Connector:XT60 -> FusIon-Pack-rescue:XT60-Connector
Changed lines of the file:
@@
 EESchema Schematic File Version 4
 LIBS:FusIon Pack-cache
-EELAYER 26 0
+EELAYER 29 0
 EELAYER END
 $Descr A4 11693 8268
@@
 $EndDescr
 $Comp
-L Connector:XT60 J5
+L FusIon-Pack-rescue:XT60-Connector J5
 U 1 1 5C4C66F7
 P 5650 3800
