File: REV 0-1 PCB/Kicad Files/POWER_STAGE.sch (KiCad schematic (older format))
At the start: 69 parts, among them Q24 IPD60N10S4L-12, Q25 IPD60N10S4L-12, Q26 IPD60N10S4L-12, Q27 IPD60N10S4L-12, Q28 IPD60N10S4L-12, Q29 IPD60N10S4L-12, Q30 IPD60N10S4L-12, Q31 IPD60N10S4L-12, Q32 IPD60N10S4L-12, Q33 IPD60N10S4L-12, Q34 FQT5P10TF, U10 BQ76200

Commit message: Fixing working tree, pushing a bunch of SubBoards and FlatPack BOM
Parts:
- Q24, Q25, Q26, Q27, Q28, Q29, Q30, Q31, Q32, Q33: symbol Transistor_FET:IPD60N10S4L-12 -> FusIon-Pack-rescue:IPD60N10S4L-12-Transistor_FET
- Q34: symbol Transistor_FET:FQT5P10TF -> FusIon-Pack-rescue:FQT5P10TF-Transistor_FET
- U10: symbol Driver_FET:BQ76200 -> FusIon-Pack-rescue:BQ76200-Driver_FET
Changed lines of the file:
@@
 EESchema Schematic File Version 4
 LIBS:FusIon Pack-cache
-EELAYER 26 0
+EELAYER 29 0
 EELAYER END
 $Descr A4 11693 8268
@@
 $EndDescr
 $Comp
-L Driver_FET:BQ76200 U10
+L FusIon-Pack-rescue:BQ76200-Driver_FET U10
 U 1 1 5D368A56
 P 4300 5650
@@
 	5050 6250 5050 6400
 $Comp
-L Transistor_FET:IPD60N10S4L-12 Q24
+L FusIon-Pack-rescue:IPD60N10S4L-12-Transistor_FET Q24
 U 1 1 5D3690F4
 P 6150 2300
@@
 $EndComp
 $Comp
-L Transistor_FET:IPD60N10S4L-12 Q25
+L FusIon-Pack-rescue:IPD60N10S4L-12-Transistor_FET Q25
 U 1 1 5D3691AA
 P 6150 2800
@@
 $EndComp
 $Comp
-L Transistor_FET:IPD60N10S4L-12 Q26
+L FusIon-Pack-rescue:IPD60N10S4L-12-Transistor_FET Q26
 U 1 1 5D369493
 P 6150 3300
@@
 $EndComp
 $Comp
-L Transistor_FET:IPD60N10S4L-12 Q27
+L FusIon-Pack-rescue:IPD60N10S4L-12-Transistor_FET Q27
 U 1 1 5D3694BB
 P 6150 3800
@@
 $EndComp
 $Comp
-L Transistor_FET:IPD60N10S4L-12 Q28
+L FusIon-Pack-rescue:IPD60N10S4L-12-Transistor_FET Q28
 U 1 1 5D3694EF
 P 6150 4300
@@
 $EndComp
 $Comp
-L Transistor_FET:IPD60N10S4L-12 Q29
+L FusIon-Pack-rescue:IPD60N10S4L-12-Transistor_FET Q29
 U 1 1 5D369553
 P 7700 2300
@@
 $EndComp
 $Comp
-L Transistor_FET:IPD60N10S4L-12 Q30
+L FusIon-Pack-rescue:IPD60N10S4L-12-Transistor_FET Q30
 U 1 1 5D369799
 P 7700 2800
@@
 $EndComp
 $Comp
-L Transistor_FET:IPD60N10S4L-12 Q31
+L FusIon-Pack-rescue:IPD60N10S4L-12-Transistor_FET Q31
 U 1 1 5D369809
 P 7700 3300
@@
 $EndComp
 $Comp
-L Transistor_FET:IPD60N10S4L-12 Q32
+L FusIon-Pack-rescue:IPD60N10S4L-12-Transistor_FET Q32
 U 1 1 5D369843
 P 7700 3800
@@
 $EndComp
 $Comp
-L Transistor_FET:IPD60N10S4L-12 Q33
+L FusIon-Pack-rescue:IPD60N10S4L-12-Transistor_FET Q33
 U 1 1 5D369877
 P 7700 4300
@@
 Connection ~ 9000 1550
 $Comp
-L Transistor_FET:FQT5P10TF Q34
+L FusIon-Pack-rescue:FQT5P10TF-Transistor_FET Q34
 U 1 1 5D4040D7
 P 7800 1650
