File: REV 0-1 PCB/Kicad Files/STM32.sch (KiCad schematic (older format))
At the start: 81 parts, among them J2 Conn_01x05_Male, Q13 RUC002N05HZGT116, Q14 RUC002N05HZGT116, SW1 SW_Push, U2 STM32F072RBTx

Commit message: Fixing working tree, pushing a bunch of SubBoards and FlatPack BOM
Parts:
- Q13, Q14: symbol Transistor_FET:RUC002N05HZGT116 -> FusIon-Pack-rescue:RUC002N05HZGT116-Transistor_FET
Changed lines of the file:
@@
 EESchema Schematic File Version 4
 LIBS:FusIon Pack-cache
-EELAYER 26 0
+EELAYER 29 0
 EELAYER END
 $Descr A4 11693 8268
@@
 POWER_BUTT
 $Comp
-L Transistor_FET:RUC002N05HZGT116 Q13
+L FusIon-Pack-rescue:RUC002N05HZGT116-Transistor_FET Q13
 U 1 1 5C765FBE
 P 3200 3350
@@
 nRST
 $Comp
-L Transistor_FET:RUC002N05HZGT116 Q14
+L FusIon-Pack-rescue:RUC002N05HZGT116-Transistor_FET Q14
 U 1 1 5C97D383
 P 3200 4300
