File: REV 0-2 PCB/FlatPack 0-2/Buck Converter SubBoard 0-2/Buck Converter SubBoard 0-2.kicad_pcb (KiCad board)
At the start: 2 copper layers, 46.4 x 25.4 mm, 33 parts, among them J1 Conn_01x04, J2 Conn_02x07_Odd_Even, U1 LMR16006, U2 ZLDO1117-33

Commit message: Fixing working tree, pushing a bunch of SubBoards and FlatPack BOM
Parts:
- R3: value 30k -> 33K
- R4: value 390R -> 1K
- R7: value 120R -> 100R
Changed lines of the file:
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@@
-(kicad_pcb (version 20171130) (host pcbnew "(5.1.2-1)-1")
+(kicad_pcb (version 20171130) (host pcbnew "(5.1.2)-2")
   (general
     (thickness 1.6)
@@
     (pad_to_mask_clearance 0.0508)
     (aux_axis_origin 0 0)
-    (visible_elements FFF9FF7F)
+    (visible_elements 7FFFFFFF)
     (pcbplotparams
-      (layerselection 0x010f0_ffffffff)
+      (layerselection 0x010fc_ffffffff)
       (usegerberextensions false)
-      (usegerberattributes true)
-      (usegerberadvancedattributes false)
+      (usegerberattributes false)
+      (usegerberadvancedattributes true)
       (creategerberjobfile false)
       (excludeedgelayer true)
@@
       (drillshape 0)
       (scaleselection 1)
-      (outputdirectory "Regulator Gerbers 6-22/"))
+      (outputdirectory "Regulator Gerbers 8-30-1649/"))
   )
   (net 0 "")
@@
       (effects (font (size 1 1) (thickness 0.15)))
     )
-    (fp_text value 30k (at 0 1.43) (layer F.Fab)
+    (fp_text value 33K (at 0 1.43) (layer F.Fab)
       (effects (font (size 1 1) (thickness 0.15)))
     )
@@
       (effects (font (size 1 1) (thickness 0.15)))
     )
-    (fp_text value 390R (at 0 1.43 180) (layer F.Fab)
+    (fp_text value 1K (at 0 1.43 180) (layer F.Fab)
       (effects (font (size 1 1) (thickness 0.15)))
     )
@@
       (effects (font (size 1 1) (thickness 0.15)))
     )
-    (fp_text value 120R (at 0 1.43 180) (layer F.Fab)
-      (effects (font (size 1 1) (thickness 0.15)))
-    )
+    (fp_text value 100R (at 0 1.43 180) (layer F.Fab)
+      (effects (font (size 1 1) (thickness 0.15)))
+    )
